File: PCB/macro-pad.kicad_pcb (KiCad board)
At the start: 2 copper layers, 116 x 88 mm, 16 parts, among them SW1 SW_Push, SW2 SW_Push, SW3 SW_Push, SW4 SW_Push, SW5 SW_Push, SW6 SW_Push, SW7 RotaryEncoder_Switch, U1 MOUDLE-SEEEDUINO-XIAO, U2 ER_OLEDM0.91_1x-I2C

Commit message: Updated the .kicad_pcb
Parts:
- moved G*** 5.36 mm to (89.0, 97.1)
Routing:
- net SWITCH_P: track 79.3 -> 87.1 mm
- net CLOCK_LINE: track 47.8 -> 48.4 mm
Other:
- board text removed: "Life is like a box of chocolates... You never know what you're gonna get. -Forrest Gump"
